File: tests/goldens/export/ecc83.kicad_pcb (KiCad board)
At the start: 2 copper layers, 40 x 30 mm, 7 parts

Commit message: carve(v0.2.0): tree export at m2-signoff
Parts:
- removed ?: , Net2Board:CP_Radial_D10.0mm_P5.00mm
- removed ?: , Net2Board:C_Disc_D4.7mm_W2.5mm_P5.00mm
- removed ?: , Net2Board:Altech_AK300_1x02_P5.00mm_45-Degree
- removed ?: , Net2Board:MountingHole_3.2mm_M3_DIN965_Pad
- removed ? (x2): , Net2Board:R_Axial_DIN0207_L6.3mm_D2.5mm_P7.62mm_Horizontal
- removed ?: , Net2Board:Valve_ECC-83-1
- added C1: , Net2Board:CP_Radial_D10.0mm_P5.00mm, F.Cu at (32.0, 6.00)
- added C2: , Net2Board:C_Disc_D4.7mm_W2.5mm_P5.00mm, B.Cu at (10.0, 20.0)
- added P1: , Net2Board:Altech_AK300_1x02_P5.00mm_45-Degree, F.Cu at (20.0, 24.0)
- added P5: , Net2Board:MountingHole_3.2mm_M3_DIN965_Pad, B.Cu at (6.00, 26.0)
- added R1: , Net2Board:R_Axial_DIN0207_L6.3mm_D2.5mm_P7.62mm_Horizontal, F.Cu at (8.00, 6.00)
- added R2: , Net2Board:R_Axial_DIN0207_L6.3mm_D2.5mm_P7.62mm_Horizontal, F.Cu at (20.0, 6.00)
- added U1: , Net2Board:Valve_ECC-83-1, F.Cu at (20.0, 14.0)
Changed lines of the file:
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@@
 		(layer "F.Cu")
 		(at 32.000000 6.000000 180)
+		(property "Reference" "C1"
+			(at 0 0 0)
+			(layer "F.SilkS")
+		)
 		(fp_circle
 			(center 2.500000 0.000000)
@@
 		(layer "B.Cu")
 		(at 10.000000 20.000000 270)
+		(property "Reference" "C2"
+			(at 0 0 0)
+			(layer "B.SilkS")
+		)
 		(fp_rect
 			(start -6.050000 -1.500000)
@@
 		(layer "F.Cu")
 		(at 20.000000 24.000000 180)
+		(property "Reference" "P1"
+			(at 0 0 0)
+			(layer "F.SilkS")
+		)
 		(fp_rect
 			(start -2.750000 -6.250000)
@@
 		(layer "B.Cu")
 		(at 6.000000 26.000000 0)
+		(property "Reference" "P5"
+			(at 0 0 0)
+			(layer "B.SilkS")
+		)
 		(fp_circle
 			(center 0.000000 0.000000)
@@
 		(layer "F.Cu")
 		(at 8.000000 6.000000 0)
+		(property "Reference" "R1"
+			(at 0 0 0)
+			(layer "F.SilkS")
+		)
 		(fp_rect
 			(start -1.050000 -1.500000)
@@
 		(layer "F.Cu")
 		(at 20.000000 6.000000 90)
+		(property "Reference" "R2"
+			(at 0 0 0)
+			(layer "F.SilkS")
+		)
 		(fp_rect
 			(start -1.050000 -1.500000)
@@
 		(layer "F.Cu")
 		(at 20.000000 14.000000 0)
+		(property "Reference" "U1"
+			(at 0 0 0)
+			(layer "F.SilkS")
+		)
 		(fp_circle
 			(center 0.000000 0.050000)

Commit message: carve(v0.3.0): tree export at m3-signoff
Changed lines of the file:
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@@
 		)
 		(pad "1" thru_hole rect
-			(at 0.000000 0.000000)
+			(at 0.000000 0.000000 180)
 			(size 2.000000 2.000000)
 			(drill 1.000000)
@@
 		)
 		(pad "2" thru_hole circle
-			(at 5.000000 0.000000)
+			(at 5.000000 0.000000 180)
 			(size 2.000000 2.000000)
 			(drill 1.000000)
@@
 		)
 		(pad "1" thru_hole circle
-			(at 0.000000 0.000000)
+			(at 0.000000 0.000000 90)
 			(size 1.600000 1.600000)
 			(drill 0.800000)
@@
 		)
 		(pad "2" thru_hole circle
-			(at -5.000000 0.000000)
+			(at -5.000000 0.000000 90)
 			(size 1.600000 1.600000)
 			(drill 0.800000)
@@
 		)
 		(pad "1" thru_hole rect
-			(at 0.000000 0.000000)
+			(at 0.000000 0.000000 180)
 			(size 3.000000 3.000000)
 			(drill 1.500000)
@@
 		)
 		(pad "2" thru_hole circle
-			(at 5.000000 0.000000)
+			(at 5.000000 0.000000 180)
 			(size 3.000000 3.000000)
 			(drill 1.500000)
@@
 		)
 		(pad "1" thru_hole circle
-			(at 0.000000 0.000000)
+			(at 0.000000 0.000000 180)
 			(size 5.600000 5.600000)
 			(drill 3.200000)
@@
 		)
 		(pad "1" thru_hole circle
-			(at 0.000000 0.000000)
+			(at 0.000000 0.000000 90)
 			(size 1.600000 1.600000)
 			(drill 0.800000)
@@
 		)
 		(pad "2" thru_hole oval
-			(at 7.620000 0.000000)
+			(at 7.620000 0.000000 90)
 			(size 1.600000 1.600000)
 			(drill 0.800000)
