File: tests/goldens/export/ecc83_acceptance.kicad_pcb (KiCad board)
At the start: 2 copper layers, 40 x 30 mm, 15 parts

Commit message: carve(v0.2.0): tree export at m2-signoff
Parts:
- removed ?: , Net2Board:CP_Radial_D10.0mm_P5.00mm
- removed ? (x4): , Net2Board:MountingHole_3.2mm_M3_DIN965_Pad
- removed ? (x4): , Net2Board:R_Axial_DIN0207_L6.3mm_D2.5mm_P7.62mm_Horizontal
- removed ?: , Net2Board:Valve_ECC-83-1
- removed ?: , Net2Board:C_Disc_D4.7mm_W2.5mm_P5.00mm
- removed ? (x4): , Net2Board:Altech_AK300_1x02_P5.00mm_45-Degree
- added C1: , Net2Board:CP_Radial_D10.0mm_P5.00mm, B.Cu at (14.0, 21.0)
- added C2: , Net2Board:C_Disc_D4.7mm_W2.5mm_P5.00mm, F.Cu at (16.2, 1.50)
- added P1: , Net2Board:Altech_AK300_1x02_P5.00mm_45-Degree, F.Cu at (1.00, 4.00)
- added P2: , Net2Board:Altech_AK300_1x02_P5.00mm_45-Degree, F.Cu at (1.00, 25.0)
- added P3: , Net2Board:Altech_AK300_1x02_P5.00mm_45-Degree, F.Cu at (39.0, 4.00)
- added P4: , Net2Board:Altech_AK300_1x02_P5.00mm_45-Degree, F.Cu at (39.0, 25.0)
- added P5: , Net2Board:MountingHole_3.2mm_M3_DIN965_Pad, F.Cu at (25.5, 1.50)
- added P6: , Net2Board:MountingHole_3.2mm_M3_DIN965_Pad, F.Cu at (33.0, 28.0)
- added P7: , Net2Board:MountingHole_3.2mm_M3_DIN965_Pad, F.Cu at (12.0, 1.50)
- added P8: , Net2Board:MountingHole_3.2mm_M3_DIN965_Pad, F.Cu at (32.0, 1.50)
- added R1: , Net2Board:R_Axial_DIN0207_L6.3mm_D2.5mm_P7.62mm_Horizontal, F.Cu at (11.0, 27.5)
- added R2: , Net2Board:R_Axial_DIN0207_L6.3mm_D2.5mm_P7.62mm_Horizontal, F.Cu at (21.0, 27.5)
- added R3: , Net2Board:R_Axial_DIN0207_L6.3mm_D2.5mm_P7.62mm_Horizontal, F.Cu at (33.4, 14.9)
- added R4: , Net2Board:R_Axial_DIN0207_L6.3mm_D2.5mm_P7.62mm_Horizontal, F.Cu at (0.50, 14.5)
- added U1: , Net2Board:Valve_ECC-83-1, F.Cu at (20.0, 15.0)
Changed lines of the file:
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@@
 		(layer "B.Cu")
 		(at 14.000000 21.000000 0)
+		(property "Reference" "C1"
+			(at 0 0 0)
+			(layer "B.SilkS")
+		)
 		(fp_circle
 			(center -2.500000 0.000000)
@@
 		(layer "F.Cu")
 		(at 16.200000 1.500000 0)
+		(property "Reference" "C2"
+			(at 0 0 0)
+			(layer "F.SilkS")
+		)
 		(fp_rect
 			(start -1.050000 -1.500000)
@@
 		(layer "F.Cu")
 		(at 1.000000 4.000000 0)
+		(property "Reference" "P1"
+			(at 0 0 0)
+			(layer "F.SilkS")
+		)
 		(fp_rect
 			(start -2.750000 -6.250000)
@@
 		(layer "F.Cu")
 		(at 1.000000 25.000000 0)
+		(property "Reference" "P2"
+			(at 0 0 0)
+			(layer "F.SilkS")
+		)
 		(fp_rect
 			(start -2.750000 -6.250000)
@@
 		(layer "F.Cu")
 		(at 39.000000 4.000000 0)
+		(property "Reference" "P3"
+			(at 0 0 0)
+			(layer "F.SilkS")
+		)
 		(fp_rect
 			(start -2.750000 -6.250000)
@@
 		(layer "F.Cu")
 		(at 39.000000 25.000000 0)
+		(property "Reference" "P4"
+			(at 0 0 0)
+			(layer "F.SilkS")
+		)
 		(fp_rect
 			(start -2.750000 -6.250000)
@@
 		(layer "F.Cu")
 		(at 25.500000 1.500000 0)
+		(property "Reference" "P5"
+			(at 0 0 0)
+			(layer "F.SilkS")
+		)
 		(fp_circle
 			(center 0.000000 0.000000)
@@
 		(layer "F.Cu")
 		(at 33.000000 28.000000 0)
+		(property "Reference" "P6"
+			(at 0 0 0)
+			(layer "F.SilkS")
+		)
 		(fp_circle
 			(center 0.000000 0.000000)
@@
 		(layer "F.Cu")
 		(at 12.000000 1.500000 0)
+		(property "Reference" "P7"
+			(at 0 0 0)
+			(layer "F.SilkS")
+		)
 		(fp_circle
 			(center 0.000000 0.000000)
@@
 		(layer "F.Cu")
 		(at 32.000000 1.500000 0)
+		(property "Reference" "P8"
+			(at 0 0 0)
+			(layer "F.SilkS")
+		)
 		(fp_circle
 			(center 0.000000 0.000000)
@@
 		(layer "F.Cu")
 		(at 11.000000 27.500000 0)
+		(property "Reference" "R1"
+			(at 0 0 0)
+			(layer "F.SilkS")
+		)
 		(fp_rect
 			(start -1.050000 -1.500000)
@@
 		(layer "F.Cu")
 		(at 21.000000 27.500000 0)
+		(property "Reference" "R2"
+			(at 0 0 0)
+			(layer "F.SilkS")
+		)
 		(fp_rect
 			(start -1.050000 -1.500000)
@@
 		(layer "F.Cu")
 		(at 33.400000 14.900000 90)
+		(property "Reference" "R3"
+			(at 0 0 0)
+			(layer "F.SilkS")
+		)
 		(fp_rect
 			(start -1.050000 -1.500000)
@@
 		(layer "F.Cu")
 		(at 0.500000 14.500000 0)
+		(property "Reference" "R4"
+			(at 0 0 0)
+			(layer "F.SilkS")
+		)
 		(fp_rect
 			(start -1.050000 -1.500000)
@@
 		(layer "F.Cu")
 		(at 20.000000 15.000000 0)
+		(property "Reference" "U1"
+			(at 0 0 0)
+			(layer "F.SilkS")
+		)
 		(fp_circle
 			(center 0.000000 0.050000)

Commit message: carve(v0.3.0): tree export at m3-signoff
Changed lines of the file:
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@@
 		)
 		(pad "1" thru_hole rect
-			(at 0.000000 0.000000)
+			(at 0.000000 0.000000 180)
 			(size 2.000000 2.000000)
 			(drill 1.000000)
@@
 		)
 		(pad "2" thru_hole circle
-			(at -5.000000 0.000000)
+			(at -5.000000 0.000000 180)
 			(size 2.000000 2.000000)
 			(drill 1.000000)
@@
 		)
 		(pad "1" thru_hole circle
-			(at 0.000000 0.000000)
+			(at 0.000000 0.000000 90)
 			(size 1.600000 1.600000)
 			(drill 0.800000)
@@
 		)
 		(pad "2" thru_hole oval
-			(at 7.620000 0.000000)
-			(size 1.600000 1.600000)
-			(drill 0.800000)
+			(at 7.620000 0.000000 90)
+			(size 1.600000 1.600000)
+			(drill 0.800000)
